Commit message: Update initial_positions_file path in bracket_arm configuration

File: config/bracket_arm.ros2_control.xacro (robot description, xacro)
@@ -2,5 +2,7 @@
 <robot xmlns:xacro="http://www.ros.org/wiki/xacro">
     <xacro:macro name="bracket_arm_ros2_control" params="name initial_positions_file">
-        <xacro:property name="initial_positions" value="${load_yaml(initial_positions_file)['initial_positions']}"/>
+        <xacro:property
+            name="initial_positions"
+            value="${load_yaml(initial_positions_file)['initial_positions']}"/>
         <ros2_control name="${name}" type="system">
             <hardware>

File: config/bracket_arm.urdf.xacro (robot description, xacro)
@@ -1,5 +1,6 @@
 <?xml version="1.0"?>
 <robot xmlns:xacro="http://www.ros.org/wiki/xacro" name="bracket_arm">
-    <xacro:arg name="initial_positions_file" default="initial_positions.yaml" />
+    <xacro:arg name="initial_positions_file"
+        default="$(find ba_arduino_controller_moveit_config)/config/initial_positions.yaml"/>
     <!-- Import bracket_arm urdf file -->
     <xacro:include filename="$(find BAArduinoController)/urdf/bracket_arm.urdf" />
